File: circuit/Device-ATmega88_Board/Device-ATmega88_Board.kicad_pcb (KiCad board)
At the start: 2 copper layers, 49.8 x 68.8 mm, 24 parts, among them J1 7seg, J2 USB_A, J3 Conn_01x06_Female, J4 Conn_01x06_Female, J5 ICSP, Q1 2SC1815, Q2 2SC1815, Q3 2SC1815, Q4 2SC1815, U1 ATmega328P-P

Commit message: プログラムを追加
Parts:
- added G***: LOGO, Meister:MeisterLogo, F.Cu at (79.0, 33.8)
Other:
- board text added: "Meister 2023"
